File: schematic/open_game_module.kicad_pcb (KiCad board)
At the start: 2 copper layers, 78.3 x 49 mm, 17 parts, among them J1 Expansion Port, J2 Conn_02x05_Odd_Even, U1 EPM7064S, U2 YMZ284, U3 HM62256BLP

Commit message: fix resistor for output to 2k2 due to internal sound chip conflict issue
Parts:
- R5: value 470R -> 2k2
Changed lines of the file:
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@@
 			)
 		)
-		(property "Value" "470R"
+		(property "Value" "2k2"
 			(at 5.08 2.37 90)
 			(layer "F.Fab")
